File: Hardware/Basic_VCO/Basic_VCO.kicad_sch (KiCad schematic)
At the start: 0 parts

Commit message: Initial Design Work - Test
Parts:
- added C1, C2: 0.1uF, symbol Device:C
- added C3, C4, C6: 10nF, symbol Device:C
- added C5: 3.9nF, symbol Device:C
- added R1, R13: 267, symbol Device:R_US
- added R10: 267k, symbol Device:R_US
- added R11: 12.7k, symbol Device:R_US
- added R12, R8: 10k, symbol Device:R_US
- added R2, R3: 20k, symbol Device:R_US
- added R4: 4.02k, symbol Device:R_US
- added R5, R6: 4.75k, symbol Device:R_US
- added R7: 49.9k, symbol Device:R_US
- added R9: 100k, symbol Device:R_US
- added RV1, RV2: 5k, symbol Device:R_Potentiometer_Trim_US
- added U1: SSI2130, Package_DFN_QFN:QFN-32-1EP_4x4mm_P0.4mm_EP2.65x2.65mm, symbol SSI:SSI2130
- added U2: TL431LP, Package_TO_SOT_THT:TO-92_Inline, symbol Reference_Voltage:TL431LP
- added U3: L78L05_TO92, Package_TO_SOT_THT:TO-92_Inline, symbol Regulator_Linear:L78L05_TO92
Connections:
- new net: R4.1, R5.1, U1.2 (SINE_IN+)
- new net: R11.1, R6.1, U1.3 (SINE_IN-)
- new net: R10.2, R7.2, R8.2, R9.1, U1.7 (EXPO_FREQ)
- new net: R10.1, RV2.2
- new net: RV2.3, U1.6 (HF_TRACK)
- new net: C6.1, R13.1
- new net: R13.2, U1.26 (BW_COMP)
- new net: C4.2, U1.19 (SOFT_SYNC)
- new net: C5.1, U1.14 (TCAP)
- new net: C3.2, U1.17 (HARD_SYNC)
- new net: R8.1, RV1.2
- new net +12V: C1.1, U3.3 (VI)
- new net +2V5: R1.2, R11.2, R9.2, RV1.1, U1.23 (VREF), U2.1 (REF), U2.3 (K)
- new net +5V: C2.1, R1.1, R2.2, U1.27 (V+), U3.1 (VO)
- new net -12V: U1.8 (V-)
- new net GND: C1.2, C2.2, C5.2, C6.2, R12.1, R3.1, R5.2, R6.2, RV1.3, RV2.1, U1.15 (DGND), U1.16 (AGND), U1.20 (HFT_BASE), U1.31 (PWM-), U2.2 (A), U3.2 (GND)
- new net HARD SYNC IN: C3.1, R12.2
- new net NOTE CV: R7.1
- new net PULSE OUT: U1.30 (PULSE_OUT)
- new net SINE OUT: U1.24 (SINE_OUT)
- new net SOFT SYNC IN: C4.1
- new net SQUARE OUT: R2.1, R3.2, U1.28 (SQUARE_OUT)
- new net TRI OUT: R4.2, U1.1 (TRI_OUT)
Other:
- title: (none) -> Basic VCO

Commit message: Update Basic_VCO.kicad_sch
Parts:
- added R14, R16: 100, symbol Device:R_US
- added R15: 19.6k, symbol Device:R_US
- added R18: 10k, symbol Device:R_US
- added RV3: 5k, symbol Device:R_Potentiometer_US
Connections:
- net +2V5: now also R18.2
- net +5V: now also R14.1
- net -12V: now also R15.2
- net GND: now also R16.2
- net PWM+: now reaches U1.32 (PWM+)
- net PWM+: now also RV3.2
- new net: R15.1, R16.1, RV3.3
- new net: R14.2, R18.1, RV3.1

Commit message: modified:   Hardware/Basic_VCO/Basic_VCO.kicad_sch
Parts:
- added R17: 10k, symbol Device:R_US
- added R19: 22.1k, symbol Device:R_US
- added RV4: 5k, symbol Device:R_Potentiometer_Trim_US
- added SW1, SW2: SW_SPDT, symbol Switch:SW_SPDT
Connections:
- net +2V5: now also R19.1
- net GND: now also R17.2
- net PWM+: now also SW1.2 (B); no longer RV3.2
- net TRI OUT: now also SW2.1 (A)
- net SAW OUT: now reaches U1.29 (SAW_OUT)
- net SAW OUT: now also SW2.3 (C)
- net LIN FREQ IN: now reaches U1.21 (LIN_FREQ)
- net at U1.22 (EXPO_SCALE): now also RV4.3
- net MIX OUT: now reaches U1.25 (MIX_OUT)
- net MIX OUT: now also R17.1
- new net: R19.2, RV4.1, RV4.2
- new net: SW1.3 (C), SW2.2 (B)
- new net PWM_1: RV3.2, SW1.1 (A)
Other:
- moved on the sheet: C3, C4, C5, C6, R10, R12, R13, R7, R8, R9, RV1, RV2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

Commit message: Updated Basic VCO schematic, still missing inputs, and mixer controls.
Parts:
- removed SW1: SW_SPDT, symbol Switch:SW_SPDT
- added C10, C12, C13, C14: 0.1u, symbol Device:C
- added C11, C7, C8: 100p, symbol Device:C
- added C9: 10u, symbol Device:C
- added Q1: 2N7000, Package_TO_SOT_THT:TO-92_Inline, symbol Transistor_FET:2N7000
- added R20, R21, R22, R23, R24, R25: 20k, symbol Device:R_US
- added R26: 499k, symbol Device:R_US
- added R27: 100, symbol Device:R_US
- added R28: 100k, symbol Device:R_US
- added R29: 10k, symbol Device:R_US
- added SW2: SW_DPDT_x2, symbol Switch:SW_DPDT_x2
- added SW3: SW_SPDT, symbol Switch:SW_SPDT
- added U1: TL072, symbol Amplifier_Operational:TL072
- added U5: LM311, symbol Comparator:LM311
- renumbered R14 to R1, R9 to R10, R5 to R11, R6 to R12, R4 to R14, R11 to R15, R19 to R16, R2 to R17, R3 to R18, R17 to R19, R16 to R2, R12 to R3, R18 to R4, R15 to R5, R7 to R6, R1 to R7, R10 to R9, RV3 to RV1, RV1 to RV2, RV2 to RV3, SW2 to SW1, U3 to U2, U2 to U3, U1 to U4
Connections:
- net PWM_1 is gone; now on net PWM+: RV1.2
- net +12V: now also C12.1, U5.8 (V+)
- net +2V5: now also R24.2, SW2.1 (A)
- net +5V: now also R29.2, SW3.1 (A)
- net -12V: now also C10.2, C13.1, C14.1, U1.4 (V-), U1.8 (V+), U5.4 (V-)
- net GND: now also C10.1, C12.2, C13.2, C14.2, Q1.1 (S), R27.1, SW3.3 (C), U1.3 (+), U5.1 (GND); no longer U4.31 (PWM-)
- net LIN FREQ IN: now also R26.2
- net PWM-: now reaches SW1.2 (B)
- net PWM-: now also U4.31 (PWM-)
- net TIME REV IN: now reaches U4.18 (TIME_REVERSE)
- net TIME REV IN: now also SW2.5 (B)
- new net: R26.1, SW2.2 (B)
- new net: C7.2, R21.2, SW2.3 (C), U1.7
- new net: C8.1, R22.1, R24.1, R25.2, U1.2 (-)
- new net: C8.2, R20.1, R22.2, R23.1, U1.1, U5.3 (-)
- new net: C7.1, R21.1, R23.2, U1.6 (-)
- new net: SW2.4 (A), SW3.2 (B)
- new net: C11.2, Q1.2 (G), R29.1, SW2.6 (C), U5.7
- new net: Q1.3 (D), R20.2, U1.5 (+)
- new net: C11.1, R28.2
- new net: R27.2, R28.1, U5.2 (+)
- new net FM IN: C9.2, R25.1
- new net PM IN: C9.1
Other:
- note added: "FM/PM Circuitry"
- note added: "Modulation Inputs"
- note added: "PWM Circuitry"
- note added: "Power Regulation/Delivery Circuitry"
- note added: "Waveform Outputs"
- moved on the sheet: C1, C2, C3, C4, C5, C6, R1, R10, R11, R12, R13, R14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
