File: Hardware/Basic_VCO/Basic_VCO.kicad_sch (KiCad schematic)
At the start: 56 parts, among them Q1 2N7000, SW1 SW_SPDT, SW2 SW_DPDT_x2, SW3 SW_SPDT, U1 TL072, U2 L78L05_TO92, U3 TL431LP, U4 SSI2130, U5 LM311

Commit message: Additional work to VCO schematic
Parts:
- removed C13, C14: 0.1u, symbol Device:C
- added C1: 0.33uF, symbol Device:C
- added C10, C13, C14, C15, C16, C17, C18, C19, C20, C7, C8, C9: 0.1uF, symbol Device:C_Small
- added C27: 100p, symbol Device:C
- added C3: 0.1uF, symbol Device:C
- added D1, D2, D3: 1N4148, Diode_THT:D_DO-35_SOD27_P7.62mm_Horizontal, symbol Diode:1N4148
- added J1, J2, J3, J4, J5, J6, J7, J8, J9: AudioJack2_SwitchT, symbol Connector_Audio:AudioJack2_SwitchT
- added R10, R11, R12, R13, R14, R18, R23, R31, R32, R38, R39, R42, R62, R63: 10k, symbol Device:R_US
- added R17: 90k, symbol Device:R_US
- added R24, R25, R26, R27, R28, R29, R30, R33, R34, R35, R40, R41, R47, R64, R65, R68: 20k, symbol Device:R_US
- added R3: 1M, symbol Device:R_US
- added R4: 267, symbol Device:R_US
- added R48, R49, R69, R70: 40k, symbol Device:R_US
- added R52, R53, R54, R71, R72, R73: 1k, symbol Device:R_US
- added R66, R67: 100k, symbol Device:R_US
- added R9: 15k, symbol Device:R_US
- added RV2, RV4, RV7: 100k, symbol Device:R_Potentiometer_US
- added SW2: SW_SPDT, symbol Switch:SW_SPDT
- added U10, U11, U3, U8: TL074, symbol Amplifier_Operational:TL074
- added U2: L78L05_TO92, Package_TO_SOT_THT:TO-92_Inline, symbol Regulator_Linear:L78L05_TO92
- added U4: TL431LP, Package_TO_SOT_THT:TO-92_Inline, symbol Reference_Voltage:TL431LP
- added U9: TL072, symbol Amplifier_Operational:TL072
- renumbered C5 to C11, C6 to C12, C1 to C2, C9 to C21, C8 to C22, C10 to C23, C7 to C24, C12 to C25, C11 to C26, C2 to C4, C3 to C5, C4 to C6, R3 to R1, R13 to R15, R1 to R19, R6 to R2, R2 to R20, R4 to R21, R5 to R22, R11 to R36, R12 to R37, R14 to R43, R15 to R44, R25 to R45, R24 to R46, R7 to R5, R22 to R50, R27 to R51, R23 to R55, R20 to R56, R28 to R57, R21 to R58, R17 to R59, R8 to R6, R18 to R60, R29 to R61, R9 to R7, R26 to R74, R19 to R75, R10 to R8, RV2 to RV1, RV4 to RV5, RV1 to RV6, SW2 to SW3, SW3 to SW4, U2 to U1, U5 to U13, U3 to U5, U1 to U6, U4 to U7
Connections:
- net +12V: now also U6.8 (V+), C13.1, C15.1, C17.1, C19.1, C7.1, C9.1, U10.4 (V+), U11.4 (V+), U3.4 (V+), U8.4 (V+), U9.8 (V+)
- net +5V: now also RV4.1
- net -12V: now also C1.1, C10.2, C14.2, C16.2, C18.2, C20.2, C8.2, U10.11 (V-), U11.11 (V-), U2.3 (VI), U3.11 (V-), U8.11 (V-), U9.4 (V-); no longer U6.8 (V+)
- net GND: now also C1.2, C10.1, C13.2, C14.1, C15.2, C16.1, C17.2, C18.1, C19.2, C20.1, C3.2, C7.2, C8.1, C9.2, J1.S, J1.TN, J2.S, J2.TN, J3.S, J3.TN, J4.S, J5.S, J6.S, J7.S, J8.S, J9.S, R10.2, R11.1, R18.1, R3.2, R33.1, R66.1, R67.1, RV2.3, RV4.3, RV7.3, U10.13 (-), U10.3 (+), U10.5 (+), U2.2 (GND), U4.1 (REF), U4.3 (K), U8.10 (+), U8.12 (+), U8.3 (+), U8.5 (+)
- net MIX OUT: now also U9.2 (-)
- net NOTE CV: now also U3.1, U3.2 (-)
- net PULSE OUT: now also R63.1
- net SAW OUT: now also R39.1
- net SINE OUT: now also R42.1
- net SQUARE OUT: now also R62.1
- net TRI OUT: now also R38.1
- net SAW MIX: now reaches U7.10 (SAW_MIX)
- net SAW MIX: now also R35.2
- net PULSE MIX: now reaches U7.11 (PULSE_MIX)
- net PULSE MIX: now also R30.1
- net at U7.12 (AUX1_MIX): now also R66.2
- net at U7.13 (AUX2_MIX): now also R67.2
- net TRI MIX: now reaches U7.9 (TRI_MIX)
- net TRI MIX: now also R27.2
- net FM IN: no longer names the net of C21.2, R45.1
- net FM IN: now also SW2.1 (A)
- net PM IN: no longer names the net of C21.1
- net PM IN: now also SW2.3 (C)
- new net: R11.2, R14.1, U11.2 (-)
- new net: R14.2, R17.1, U11.1
- new net: R38.2, R40.2, R48.2, U8.2 (-)
- new net: R32.2, R33.2, U10.10 (+)
- new net: R34.2, R35.1, U10.8
- new net: R31.1, R34.1, U10.9 (-)
- new net: R13.1, RV4.2
- new net: R12.2, R13.2, U11.3 (+)
- new net: J1.T, R3.1, U3.3 (+)
- new net: J6.T, R54.1
- new net: R47.1, R54.2, U10.14
- new net: R29.2, R30.2, R31.2, U10.7
- new net: R23.2, R24.2, R25.1, R26.1, R32.1, U10.2 (-)
- new net: J8.T, R72.1
- new net: R69.1, R72.2, U8.8
- new net: D3.2 (A), R26.2, R28.1
- new net: R28.2, R29.1, U10.6 (-)
- new net: J2.T, RV2.1
- new net: R17.2, R18.2, U11.5 (+)
- new net: RV7.2, U11.10 (+)
- new net: D1.1 (K), RV7.1, U11.6 (-)
- new net: D1.2 (A), U11.7
- new net: R39.2, R41.2, R49.2, U8.6 (-)
- new net: D2.1 (K), R25.2, R27.1
- new net: D2.2 (A), D3.1 (K), U10.1
- new net: RV2.2, U3.5 (+)
- new net: R63.2, R65.2, R70.2, U8.13 (-)
- new net: J5.T, R53.1
- new net: R49.1, R53.2, U8.7
- new net: C27.2, R68.2, R71.1, U9.1
- new net: C27.1, R68.1, U9.3 (+)
- new net: R48.1, R52.2, U8.1
- new net: R62.2, R64.2, R69.2, U8.9 (-)
- new net: R42.2, R47.2, U10.12 (+)
- new net: J9.T, R73.1
- new net: R70.1, R73.2, U8.14
- new net: J4.T, R52.1
- new net: R10.1, R9.2, U9.5 (+)
- new net: J3.T, R12.1
- new net: J7.T, R71.2
- new net -1V: R24.1, U9.6 (-), U9.7
- new net -2V5: R4.2, R40.1, R41.1, R64.1, R65.1, R9.1, U4.2 (A)
- new net -5V: C3.1, R4.1, U2.1 (VO)
- new net CROSSFADE CV: R23.1, U11.8, U11.9 (-)
- new net PM/FM IN: SW2.2 (B), U3.6 (-), U3.7
- no-connect marks 0 -> 10
Other:
- note added: "CROSSFADE MIXER"
- note added: "FM/PM"
- note added: "PWM"
- note added: "Power Regulation/Delivery"
- note added: "Waveform Outputs + Mixer In/Out"
- note removed: "FM/PM Circuitry"
- note removed: "PWM Circuitry"
- note removed: "Power Regulation/Delivery Circuitry"
- note removed: "Waveform Outputs"
- moved on the sheet: C11, C12, C2, C21, C22, C23, C24, C25, C26, C4, C5, C6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

Commit message: Finished 1st revision schematic for Basic VCO
Parts:
- removed U2: L78L05_TO92, Package_TO_SOT_THT:TO-92_Inline, symbol Regulator_Linear:L78L05_TO92
- added D1, D2, D3, D4: 1N5817, Diode_THT:D_DO-41_SOD81_P10.16mm_Horizontal, symbol Diode:1N5817
- added J3, J5: AudioJack2_SwitchT, symbol Connector_Audio:AudioJack2_SwitchT
- added J6: Conn_02x05_Odd_Even, symbol Connector_Generic:Conn_02x05_Odd_Even
- added R1, R2: 10, symbol Device:R_US
- added R21, R23, R5, R7: 49.9k, symbol Device:R_US
- added U2: L79L05_SOT89, Package_TO_SOT_SMD:SOT-89-3, symbol Regulator_Linear:L79L05_SOT89
- C1: renamed from C2; value 0.1uF -> 0.33uF
- R15: renamed from R11; value 10k -> 49.9k
- R16: renamed from R12; value 10k -> 49.9k
- R17: renamed from R13; value 10k -> 49.9k
- R18: renamed from R14; value 10k -> 49.9k
- R22: renamed from R17; value 90k -> 90.9k
- R54: renamed from R48; value 40k -> 40.2k
- R55: renamed from R49; value 40k -> 40.2k
- R75: renamed from R69; value 40k -> 40.2k
- R76: renamed from R70; value 40k -> 40.2k
- renumbered C1 to C2, C4 to C3, C3 to C4, D1 to D5, D2 to D6, D3 to D7, J7 to J10, J8 to J11, J9 to J12, J3 to J4, J4 to J7, J5 to J8, J6 to J9, R4 to R10, R7 to R11, R8 to R12, R9 to R13, R10 to R14, R15 to R19, R16 to R20, R18 to R24, R19 to R25, R20 to R26, R21 to R27, R22 to R28, R23 to R29, R1 to R3, R24 to R30, R25 to R31, R26 to R32, R27 to R33, R28 to R34, R29 to R35, R30 to R36, R31 to R37, R32 to R38, R33 to R39, R2 to R4, R34 to R40, R35 to R41, R36 to R42, R37 to R43, R38 to R44, R39 to R45, R40 to R46, R41 to R47, R42 to R48, R43 to R49, R44 to R50, R45 to R51, R46 to R52, R47 to R53, R50 to R56, R51 to R57, R52 to R58, R53 to R59, R3 to R6, R54 to R60, R55 to R61, R56 to R62, R57 to R63, R58 to R64, R59 to R65, R60 to R66, R61 to R67, R62 to R68, R63 to R69, R64 to R70, R65 to R71, R66 to R72, R67 to R73, R68 to R74, R71 to R77, R72 to R78, R73 to R79, R5 to R8, R74 to R80, R75 to R81, R6 to R9, U13 to U12, U5 to U4, U4 to U5
Connections:
- net +12V: now also J6.10 (Pin_10), J6.9 (Pin_9), R1.1; no longer C1.1, U1.3 (VI)
- net +2V5: now also D1.1 (K), D3.1 (K)
- net -12V: now also J6.1 (Pin_1), J6.2 (Pin_2), R2.1; no longer C2.1
- net -5V: now also U2.3 (VO)
- net CROSSFADE CV: now also R38.1
- net GND: now also U11.13 (-), D2.2 (A), D4.2 (A), J3.S, J3.TN, J5.S, J5.TN, J6.3 (Pin_3), J6.4 (Pin_4), J6.5 (Pin_5), J6.6 (Pin_6), J6.7 (Pin_7), J6.8 (Pin_8), R23.2, R7.2, U2.1 (GND)
- net HARD SYNC IN: now also U3.13 (-), U3.14
- net SOFT SYNC IN: now also U3.8, U3.9 (-)
- net at R29.2, R30.2, R31.1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: no longer R38.1
- net at U11.12 (+): now also U11.14
- net at U3.12 (+): now also D3.2 (A), D4.1 (K), R21.2, R23.1
- net at U3.10 (+): now also D1.2 (A), D2.1 (K), R5.2, R7.1
- new net: C1.1, R1.2, U1.3 (VI)
- new net: C2.1, R2.2, U2.2 (VI)
- new net: J5.T, R21.1
- new net: J3.T, R5.1
Other:
- note added: "Adjust magnitude"
- note added: "Inputs"
- note added: "Offset input wave"
- moved on the sheet: C1, C11, C12, C2, C21, C22, C23, C24, C25, C26, C27, C3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
