File: Hardware/Basic_VCO/Basic_VCO.kicad_sch (KiCad schematic)
At the start: 151 parts, among them J1 AudioJack2_SwitchT, J10 AudioJack2_SwitchT, J11 AudioJack2_SwitchT, J12 AudioJack2_SwitchT, J2 AudioJack2_SwitchT, J3 AudioJack2_SwitchT, J4 AudioJack2_SwitchT, J5 AudioJack2_SwitchT, J6 Conn_02x05_Odd_Even, J7 AudioJack2_SwitchT, J8 AudioJack2_SwitchT, J9 AudioJack2_SwitchT, Q1 2N7000, SW1 SW_SPDT, SW2 SW_SPDT, SW3 SW_DPDT_x2, SW4 SW_SPDT, U1 L78L05_TO92, U10 TL074, U11 TL074, U12 LM311, U2 L79L05_SOT89, U3 TL074, U4 TL431LP, U5 TL431LP, U6 TL072, U7 SSI2130, U8 TL074, U9 TL072

Commit message: set some pcb footprints
Parts:
- C1, C10, C11, C12, C13, C14, C15, C16, C17, C18, C19, C2, C20, C21, C22, C23, C24, C25, C26, C27, C3, C4, C5, C6, C7, C8, C9: footprint (none) -> Capacitor_SMD:C_0402_1005Metric
- D1, D2, D3, D4: footprint Diode_THT:D_DO-41_SOD81_P10.16mm_Horizontal -> Diode_SMD:D_SOD-123
- D5, D6, D7: footprint Diode_THT:D_DO-35_SOD27_P7.62mm_Horizontal -> Diode_SMD:D_SOD-123
- Q1: footprint Package_TO_SOT_THT:TO-92_Inline -> Package_TO_SOT_SMD:SOT-23
- R1, R10, R11, R12, R13, R14, R15, R16, R17, R18, R19, R2, R20, R21, R22, R23, R24, R25, R26, R27, R28, R29, R3, R30, R31, R32, R33, R34, R35, R36, R37, R38, R39, R4, R40, R41, R42, R43, R44, R45, R46, R47, R48, R49, R5, R50, R51, R52, R53, R54, R55, R56, R57, R58, R59, R6, R60, R61, R62, R63, R64, R65, R66, R67, R68, R69, R7, R70, R71, R72, R73, R74, R75, R76, R77, R78, R79, R8, R80, R81, R9: footprint (none) -> Resistor_SMD:R_0402_1005Metric
- U10, U11, U3, U8: footprint (none) -> Package_SO:SOIC-14_3.9x8.7mm_P1.27mm
- U12, U6, U9: footprint (none) -> Package_SO:SOIC-8_3.9x4.9mm_P1.27mm
- U4, U5: footprint Package_TO_SOT_THT:TO-92_Inline -> Package_TO_SOT_SMD:SOT-23-3
- U7: footprint Package_DFN_QFN:QFN-32-1EP_4x4mm_P0.4mm_EP2.65x2.65mm -> Package_DIP:DIP-32_W15.24mm

Commit message: Changed Crossfade CV input to have 5V when disconnected instead of ground.
Previously the Crossfade CV input would be grounded when disconnected from a CV source. now it is 5V allowing it to be set statically using offset and magnitude. CV input was designed expecting 10Vp-p (+/-5V or 0-10V)  so should be fine.
Parts:
- removed unit 1 of U9
- added unit 2 of U9
Connections:
- net +5V: now also J4.TN
- net GND: now also U9.5 (+); no longer J4.TN, U11.13 (-)
- net MIX OUT: now also U11.13 (-)
- net at U11.12 (+): now also C27.1, R74.1; no longer U11.14
- net at C27.2, R74.2, R77.1: now also U11.14
- net at R13.2, R14.1: now also U9.3 (+); no longer U9.5 (+)
- removed net -1V: R30.1, U9.6 (-), U9.7
- new net: U9.6 (-), U9.7
- new net -1V0: R30.1, U9.1, U9.2 (-)
Other:
- moved on the sheet: C17, C18, D6, D7, J6, R29, R30, R31, R32, R33, R34, R35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

Commit message: adjusted schematic and prepared footprints for pcb design
Parts:
- added C28, C29: 0.1uF, Capacitor_SMD:C_0402_1005Metric, symbol Device:C_Small
- added unit 5 of U13
- added unit 4 of U13
- added unit 4 of U7
- J1, J10, J11, J12, J2, J3, J4, J5, J7, J8, J9: footprint (none) -> Connector_Audio:Jack_3.5mm_QingPu_WQP-PJ398SM_Vertical_CircularHoles
- J6: footprint (none) -> Connector_IDC:IDC-Header_2x05_P2.54mm_Vertical
- R23: renamed from R66; value 20k -> 21
- RT1: renamed from RV1; footprint (none) -> Bourns PV36Y:TRIM_PV36Y502C01B00
- RT2: renamed from RV3; footprint (none) -> Bourns PV36Y:TRIM_PV36Y502C01B00
- RT3: renamed from RV5; footprint (none) -> Bourns PV36Y:TRIM_PV36Y502C01B00
- RV1: renamed from RV2; footprint (none) -> Potentiometer_THT:Potentiometer_Alpha_RD901F-40-00D_Single_Vertical
- RV2: renamed from RV4; footprint (none) -> Potentiometer_THT:Potentiometer_Alpha_RD901F-40-00D_Single_Vertical
- RV3: renamed from RV6; footprint (none) -> Potentiometer_THT:Potentiometer_Alpha_RD901F-40-00D_Single_Vertical
- RV4: renamed from RV7; footprint (none) -> Potentiometer_THT:Potentiometer_Alpha_RD901F-40-00D_Single_Vertical
- SW1, SW2, SW4: footprint (none) -> toggleswitches:SW_100SP1T1B4M2QE
- SW3: footprint (none) -> AN12SECQE:SW6_ANT21SECQE_CRS
- U10: renamed from U11; value TL074 -> TL072; footprint Package_SO:SOIC-14_3.9x8.7mm_P1.27mm -> Package_SO:SOIC-8_3.9x4.9mm_P1.27mm; symbol Amplifier_Operational:TL074 -> Amplifier_Operational:TL072
- U10: value TL074 -> TL072; footprint Package_SO:SOIC-14_3.9x8.7mm_P1.27mm -> Package_SO:SOIC-8_3.9x4.9mm_P1.27mm; symbol Amplifier_Operational:TL074 -> Amplifier_Operational:TL072
- U2: renamed from U1; footprint Package_TO_SOT_THT:TO-92_Inline -> Package_TO_SOT_SMD:SOT-89-3
- U6: renamed from U10; value TL074 -> TL072; footprint Package_SO:SOIC-14_3.9x8.7mm_P1.27mm -> Package_SO:SOIC-8_3.9x4.9mm_P1.27mm; symbol Amplifier_Operational:TL074 -> Amplifier_Operational:TL072
- renumbered C22 to C10, C24 to C11, C25 to C12, C26 to C13, C23 to C14, C27 to C15, C7 to C16, C8 to C17, C9 to C18, C10 to C19, C3 to C2, C13 to C20, C14 to C21, C15 to C22, C16 to C23, C19 to C24, C20 to C25, C17 to C26, C18 to C27, C2 to C3, C11 to C7, C12 to C8, C21 to C9, D6 to D1, D7 to D2, D1 to D3, D2 to D4, D3 to D5, D4 to D6, D5 to D7, R9 to R10, R12 to R11, R20 to R12, R19 to R13, R25 to R14, R27 to R15, R26 to R16, R28 to R17, R42 to R18, R49 to R19, R8 to R2, R43 to R20, R50 to R21, R65 to R22, R72 to R24, R73 to R25, R81 to R26, R51 to R27, R52 to R28, R56 to R29, R2 to R3, R61 to R30, R62 to R31, R64 to R32, R57 to R33, R63 to R34, R67 to R35, R80 to R36, R29 to R37, R31 to R38, R33 to R39, R10 to R4, R30 to R40, R32 to R41, R34 to R42, R35 to R43, R36 to R44, R37 to R45, R40 to R46, R38 to R47, R39 to R48, R41 to R49, R13 to R5, R21 to R50, R23 to R51, R16 to R52, R17 to R53, R15 to R54, R18 to R55, R22 to R56, R24 to R57, R44 to R59, R14 to R6, R46 to R60, R54 to R61, R58 to R62, R45 to R63, R47 to R64, R55 to R65, R59 to R66, R68 to R67, R70 to R68, R75 to R69, R3 to R7, R78 to R70, R69 to R71, R71 to R72, R76 to R73, R79 to R74, R48 to R75, R53 to R76, R60 to R77, R74 to R78, R77 to R79, R4 to R8, R6 to R80, R5 to R81, R7 to R82, R11 to R9, U7 to U1, U9 to U10, U12 to U11, U9 to U12, U6 to U12, U10 to U13, U4 to U3, U2 to U4, U11 to U7, U3 to U7, U3 to U8, U11 to U9, U8 to U9
Connections:
- net +12V: now also U6.8 (V+), C28.1, U13.4 (V+); no longer U6.4 (V+)
- net +2V5: now also RT1.3; no longer RT1.1
- net +5V: now also RV2.3; no longer RV2.1
- net -12V: now also U6.4 (V-), C29.2, U13.11 (V-); no longer U6.11 (V-)
- net GND: now also RT1.1, RV1.1, RV2.1, RV4.1, U10.2 (-), C28.2, C29.1, U13.12 (+), U7.12 (+); no longer RT1.3, RV1.3, RV2.3, RV4.3, U10.13 (-)
- net MIX OUT: now also U10.6 (-); no longer U10.13 (-)
- net at R12.2, RT3.2: now also RT3.3; no longer RT3.1
- net at U1.22 (EXPO_SCALE): now also RT3.1; no longer RT3.3
- net at R16.1, R17.1: now also RV3.1; no longer RV3.3
- net at R76.1, R77.2: now also U10.1; no longer U10.14
- net at C15.1, R78.1: now also U10.5 (+); no longer U10.12 (+)
- net at C15.2, R78.2, R79.1: now also U10.7; no longer U10.14
- net at J2.T: now also RV1.3; no longer RV1.1
- net at D7.1 (K), U7.6 (-): now also RV4.3; no longer RV4.1
- net at R14.2, R15.1: now also RV3.3; no longer RV3.1
- net at R75.2, R76.2: now also U10.3 (+); no longer U10.12 (+)
- new net: U13.13 (-), U13.14
- new net: U7.13 (-), U7.14
Other:
- moved on the sheet: C10, C11, C12, C13, C14, C15, C5, C6, C7, C8, C9, D1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
